File: HBridgeShield/HBridgeShield.brd (EAGLE design)
At the start: 53 x 59.7 mm, 5 parts, among them X1 22-23-2041

Commit message: No deadly power connection
Connections:
- net GND: no longer J1.2
Changed lines of the file:
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@@
 </signal>
 <signal name="GND">
-<contactref element="J1" pad="2"/>
 <contactref element="J1" pad="3"/>
 <contactref element="ZX1" pad="4"/>

Commit message: Added 12v connection to Arduino board VIN
Connections:
- net 12V: now also B1.VIN
Routing:
- net 12V: track 47.9 -> 75.2 mm
Changed lines of the file:
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@@
 <wire x1="24.13" y1="40.64" x2="27.94" y2="36.83" width="0.508" layer="1"/>
 <wire x1="27.94" y1="36.83" x2="27.94" y2="17.78" width="0.508" layer="1"/>
-<wire x1="32.46" y1="13.26" x2="44.45" y2="13.26" width="0.508" layer="1"/>
+<wire x1="44.45" y1="13.26" x2="32.46" y2="13.26" width="0.508" layer="1"/>
 <wire x1="27.94" y1="17.78" x2="32.46" y2="13.26" width="0.508" layer="1"/>
+<contactref element="B1" pad="VIN"/>
+<wire x1="50.8" y1="36.83" x2="48.895" y2="36.83" width="0.4064" layer="1"/>
+<wire x1="48.895" y1="36.83" x2="47.625" y2="35.56" width="0.4064" layer="1"/>
+<wire x1="47.625" y1="35.56" x2="47.625" y2="16.435" width="0.4064" layer="1"/>
+<wire x1="47.625" y1="16.435" x2="44.45" y2="13.26" width="0.4064" layer="1"/>
 </signal>
 <signal name="GND">
